Commit message: Update mecanum drive controller configuration

File: src/my_bot/description/gazebo_control.xacro (robot description, xacro)
@@ -6,12 +6,11 @@
             <odometryTopic>odom</odometryTopic>
             <odometryRate>20.0</odometryRate>
-            <robotBaseFrame>base_footprint</robotBaseFrame>
             <!-- Wheel Information -->
-            <left_joint>back_left_wheel_joint</left_joint>
-            <right_joint>back_right_wheel_joint</right_joint>
-            <left_joint>front_right_wheel_joint</left_joint>
-            <right_joint>front_left_wheel_joint</right_joint>
-            <wheel_separation>0.35</wheel_separation>
-            <wheel_diameter>0.1</wheel_diameter>
+            <front_left_joint>front_left_wheel_joint</front_left_joint>
+            <front_right_joint>front_right_wheel_joint</front_right_joint>
+            <back_left_joint>back_left_wheel_joint</back_left_joint>
+            <back_right_joint>back_right_wheel_joint</back_right_joint>
+            <wheel_separation>0.19</wheel_separation>
+            <wheel_diameter>0.03</wheel_diameter>
             <!-- Limits -->
             <max_wheel_torque>200</max_wheel_torque>
@@ -25,32 +24,4 @@
             <publish_wheel_tf>true</publish_wheel_tf>
         </plugin>
-        <!-- <plugin name="imu_plugin" filename="libgazebo_ros_imu.so">
-            <alwaysOn>true</alwaysOn>
-            <! <bodyName>base_footprint</bodyName> >
-            <topicName>imu</topicName>
-            <serviceName>imu_service</serviceName>
-            <gaussianNoise>0.0</gaussianNoise>
-            <updateRate>20.0</updateRate>
-        </plugin> -->
-    </gazebo>
-        <gazebo reference="imu_link">
-            <gravity>false</gravity>
-            <sensor name="imu_sensor" type="imu">
-                <always_on>true</always_on>
-                <update_rate>100</update_rate>
-                <visualize>true</visualize>
-                <topic>__default_topic__</topic>
-                <plugin filename="libgazebo_ros_imu_sensor.so" name="imu_plugin">
-                    <topicName>imu</topicName>
-                    <bodyName>imu_link</bodyName>
-                    <updateRateHZ>10.0</updateRateHZ>
-                    <gaussianNoise>0.0</gaussianNoise>
-                    <xyzOffset>0 0 0</xyzOffset>
-                    <rpyOffset>0 0 0</rpyOffset>
-                    <frameName>imu_link</frameName>
-                    <initialOrientationAsReference>false</initialOrientationAsReference>
-                </plugin>
-                <pose>0 0 0 0 0 0</pose>
-            </sensor>
     </gazebo>
 </robot>

File: src/my_bot/description/lidar.xacro (robot description, xacro)
@@ -4,10 +4,10 @@
         <parent link="chassis"/>
         <child link="laser_frame"/>
-        <origin xyz="0.1 0 0.055" rpy="0 0 0"/>
+        <origin xyz="0.1 0 0.05" rpy="0 0 0"/>
     </joint>
     <link name="laser_frame">
         <visual>
             <geometry>
-                <cylinder radius="0.03" length="0.04"/>
+                <cylinder radius="0.05" length="0.04"/>
             </geometry>
             <material name="red"/>
@@ -18,10 +18,10 @@
             </geometry>
         </collision>
-        <xacro:inertial_cylinder mass="0.1" length="0.04" radius="0.03">
+        <xacro:inertial_cylinder mass="0.1" length="0.04" radius="0.05">
             <origin xyz="0 0 0" rpy="0 0 0"/>
         </xacro:inertial_cylinder>
     </link>
     <gazebo reference="laser_frame">
-        <material>Gazebo/orange</material>
+        <material>Gazebo/Red</material>
         <sensor name="laser" type="ray">
             <pose> 0 0 0 0 0 0 </pose>

File: src/my_bot/description/robot.urdf.xacro (robot description, xacro)
@@ -1,9 +1,6 @@
 <?xml version="1.0"?>
-<robot xmlns:xacro="http://www.ros.org/wiki/xacro" name="robot">
-    <!-- Include files with absolute paths -->
-    <xacro:include filename="$(find my_bot)/description/robot_core.xacro" />
-   <xacro:include filename="$(find my_bot)/description/ros2_control.xacro" />
-    <xacro:include filename="$(find my_bot)/description/lidar.xacro" />
-    <!-- Call the robot_control macro (we found this one)
-    <xacro:robot_control name="robot_control" /> -->
+<robot xmlns:xacro="http://www.ros.org/wiki/xacro"  name="robot">
+    <xacro:include filename="robot_core.xacro" />
+    <xacro:include filename="inertial_macros.xacro" />
+    <xacro:include filename="ros2_control.xacro" />
 </robot>

File: src/my_bot/description/robot_core.xacro (robot description, xacro)
@@ -14,4 +14,7 @@
         <color rgba="0 0 0 1" />
     </material>
+    <material name="red">
+        <color rgba="1 0 0 1" />
+    </material>
     <!-- BASE LINK -->
     <link name="base_link">
@@ -19,23 +22,24 @@
     <!-- CHASSIS LINK -->
     <joint name="chassis_joint" type="fixed">
-        <parent link="base_link" />
-        <child link="chassis" />
-        <origin xyz="0 0 0.023" rpy="0 0 0" />
+        <parent link="base_link"/>
+        <child link="chassis"/>
+        <origin xyz="0 0 0"/>
     </joint>
     <link name="chassis">
         <visual>
+            <origin xyz="0 0 0.1125"/>
             <geometry>
-                <box size="0.26 0.15 0.065" />
+                <box size="0.7 1 0.225"/>
             </geometry>
-            <material name="white" />
+            <material name="white"/>
         </visual>
         <collision>
-            <origin xyz="0 0 0.0325" />
+            <origin xyz="0 0 0.1125"/>
             <geometry>
-                <box size="0.26 0.15 0.065" />
+                <box size="0.7 1.0 0.225"/>
             </geometry>
         </collision>
-        <xacro:inertial_box mass="0.5" x="0.26" y="0.15" z="0.065">
-            <origin xyz="0 0 0.0325" rpy="0 0 0" />
+        <xacro:inertial_box mass="0.5" x="0.7" y="1.0" z="0.225">
+            <origin xyz="0 0 0.1125" rpy="0 0 0" />
         </xacro:inertial_box>
     </link>
@@ -45,38 +49,25 @@
     <!-- LEFT WHEEL LINK -->
     <joint name="back_left_wheel_joint" type="continuous">
-        <parent link="base_link" />
-        <child link="left_wheel" />
-        <origin xyz="-0.08 -0.095 -0.015" rpy="-${pi/2} 0 0" />
-        <axis xyz="0 0 1" />
-        <dynamics damping="0.5" friction="1.0" />
+        <parent link="base_link"/>
+        <child link="left_wheel"/>
+        <origin xyz="0.25 0.525 0" rpy="-${pi/2} 0 0" />
+        <axis xyz="0 0 1"/>
     </joint>
     <link name="left_wheel">
         <visual>
             <geometry>
-                <cylinder radius="0.03" length="0.01" />
+                <cylinder radius="0.076" length="0.04"/>
             </geometry>
-            <material name="blue" />
+            <material name="blue"/>
         </visual>
         <collision>
             <geometry>
-                <cylinder radius="0.03" length="0.01" />
+                <cylinder radius="0.076" length="0.04"/>
             </geometry>
         </collision>
-        <xacro:inertial_cylinder mass="0.1" length="0.03" radius="0.03">
+        <xacro:inertial_cylinder mass="0.5" length="0.04" radius="0.076">
             <origin xyz="0 0 0" rpy="0 0 0" />
         </xacro:inertial_cylinder>
     </link>
-    <!--
-    <transmission name="back_left_wheel_trans">
-        <type>transmission_interface/SimpleTransmission</type>
-        <joint name="back_left_wheel_joint">
-            <hardwareInterface>hardware_interface/VelocityJointInterface</hardwareInterface>
-        </joint>
-        <actuator name="back_left_wheel_motor">
-            <hardwareInterface>hardware_interface/VelocityJointInterface</hardwareInterface>
-            <mechanicalReduction>1</mechanicalReduction>
-        </actuator>
-    </transmission>
--->
     <gazebo reference="left_wheel">
         <material>Gazebo/Blue</material>
@@ -84,37 +75,25 @@
     <!-- RIGHT WHEEL LINK -->
     <joint name="back_right_wheel_joint" type="continuous">
-        <parent link="base_link" />
-        <child link="right_wheel" />
-        <origin xyz="-0.08 0.095 -0.015" rpy="${pi/2} 0 0" />
-        <axis xyz="0 0 1" />
-        <dynamics damping="0.5" friction="1.0" />
+        <parent link="base_link"/>
+        <child link="right_wheel"/>
+        <origin xyz="0.25 -0.525 0" rpy="${pi/2} 0 0" />
+        <axis xyz="0 0 -1"/>
     </joint>
     <link name="right_wheel">
         <visual>
             <geometry>
-                <cylinder radius="0.03" length="0.01" />
+                <cylinder radius="0.076" length="0.04"/>
             </geometry>
-            <material name="blue" />
+            <material name="blue"/>
         </visual>
         <collision>
             <geometry>
-                <cylinder radius="0.03" length="0.01" />
+                <cylinder radius="0.076" length="0.04"/>
             </geometry>
         </collision>
-        <xacro:inertial_cylinder mass="0.1" length="0.03" radius="0.03">
+        <xacro:inertial_cylinder mass="0.5" length="0.04" radius="0.076">
             <origin xyz="0 0 0" rpy="0 0 0" />
         </xacro:inertial_cylinder>
     </link>
-    <!--    <transmission name="back_right_wheel_trans">
-        <type>transmission_interface/SimpleTransmission</type>
-        <joint name="back_right_wheel_joint">
-            <hardwareInterface>hardware_interface/VelocityJointInterface</hardwareInterface>
-        </joint>
-        <actuator name="back_right_wheel_motor">
-            <hardwareInterface>hardware_interface/VelocityJointInterface</hardwareInterface>
-            <mechanicalReduction>1</mechanicalReduction>
-        </actuator>
-    </transmission>
--->
     <gazebo reference="right_wheel">
         <material>Gazebo/Blue</material>
@@ -124,12 +103,11 @@
         <parent link="base_link" />
         <child link="right_front_wheel" />
-        <origin xyz="0.08 0.095 -0.015" rpy="${pi/2} 0 0" />
-        <axis xyz="0 0 1" />
-        <dynamics damping="0.5" friction="1.0" />
+        <origin xyz="-0.25 -0.525 0" rpy="${pi/2} 0 0" />
+        <axis xyz="0 0 -1" />
     </joint>
     <link name="right_front_wheel">
         <visual>
             <geometry>
-                <cylinder radius="0.03" length="0.01" />
+                <cylinder radius="0.076" length="0.04" />
             </geometry>
             <material name="blue" />
@@ -137,23 +115,11 @@
         <collision>
             <geometry>
-                <cylinder radius="0.03" length="0.01" />
+                <cylinder radius="0.076" length="0.04" />
             </geometry>
         </collision>
-        <xacro:inertial_cylinder mass="0.1" length="0.03" radius="0.03">
+        <xacro:inertial_cylinder mass="0.5" length="0.04" radius="0.076">
             <origin xyz="0 0 0" rpy="0 0 0" />
         </xacro:inertial_cylinder>
     </link>
-<!--
-    <transmission name="front_right_wheel_trans">
-        <type>transmission_interface/SimpleTransmission</type>
-        <joint name="front_right_wheel_joint">
-            <hardwareInterface>hardware_interface/VelocityJointInterface</hardwareInterface>
-        </joint>
-        <actuator name="front_right_wheel_motor">
-            <hardwareInterface>hardware_interface/VelocityJointInterface</hardwareInterface>
-            <mechanicalReduction>1</mechanicalReduction>
-        </actuator>
-    </transmission>
--->
     <gazebo reference="right_front_wheel">
         <material>Gazebo/Blue</material>
@@ -163,12 +129,11 @@
         <parent link="base_link" />
         <child link="left_front_wheel" />
-        <origin xyz="0.08 -0.095 -0.015" rpy="-${pi/2} 0 0" />
+        <origin xyz="-0.25 0.525 0" rpy="-${pi/2} 0 0" />
         <axis xyz="0 0 1" />
-        <dynamics damping="0.5" friction="1.0" />
     </joint>
     <link name="left_front_wheel">
         <visual>
             <geometry>
-                <cylinder radius="0.03" length="0.01" />
+                <cylinder radius="0.076" length="0.04" />
             </geometry>
             <material name="blue" />
@@ -176,23 +141,11 @@
         <collision>
             <geometry>
-                <cylinder radius="0.03" length="0.01" />
+                <cylinder radius="0.076" length="0.04" />
             </geometry>
         </collision>
-        <xacro:inertial_cylinder mass="0.1" length="0.03" radius="0.03">
+        <xacro:inertial_cylinder mass="0.5" length="0.04" radius="0.076">
             <origin xyz="0 0 0" rpy="0 0 0" />
         </xacro:inertial_cylinder>
     </link>
-<!--
-    <transmission name="front_left_wheel_trans">
-        <type>transmission_interface/SimpleTransmission</type>
-        <joint name="front_left_wheel_joint">
-            <hardwareInterface>hardware_interface/VelocityJointInterface</hardwareInterface>
-        </joint>
-        <actuator name="front_left_wheel_motor">
-            <hardwareInterface>hardware_interface/VelocityJointInterface</hardwareInterface>
-            <mechanicalReduction>1</mechanicalReduction>
-        </actuator>
-    </transmission>
--->
     <gazebo reference="left_front_wheel">
         <material>Gazebo/Blue</material>
@@ -216,40 +169,10 @@
             </geometry>
         </collision>
-        <xacro:inertial_box mass="0.5" x="0.01" y="0.01" z="0.01">
+        <xacro:inertial_box mass="0.1" x="0.01" y="0.01" z="0.01">
             <origin xyz="0 0 0" rpy="0 0 0" />
         </xacro:inertial_box>
     </link>
-    <!-- Mecanum Wheel Friction Parameters -->
-    <gazebo reference="left_front_wheel">
-    <mu1>1.0</mu1>
-    <mu2>1.0</mu2>
-    <kp>1000000.0</kp>
-    <kd>1.0</kd>
-    <minDepth>0.001</minDepth>
-    <maxVel>1.0</maxVel>
-</gazebo>
-<gazebo reference="right_front_wheel">
-    <mu1>1.0</mu1>
-    <mu2>1.0</mu2>
-    <kp>1000000.0</kp>
-    <kd>1.0</kd>
-    <minDepth>0.001</minDepth>
-    <maxVel>1.0</maxVel>
-</gazebo>
-<gazebo reference="left_wheel">
-    <mu1>1.0</mu1>
-    <mu2>1.0</mu2>
-    <kp>1000000.0</kp>
-    <kd>1.0</kd>
-    <minDepth>0.001</minDepth>
-    <maxVel>1.0</maxVel>
-</gazebo>
-<gazebo reference="right_wheel">
-    <mu1>1.0</mu1>
-    <mu2>1.0</mu2>
-    <kp>1000000.0</kp>
-    <kd>1.0</kd>
-    <minDepth>0.001</minDepth>
-    <maxVel>1.0</maxVel>
-</gazebo>
+    <gazebo reference="imu_link">
+        <material>Gazebo/White</material>
+    </gazebo>
 </robot>

File: src/my_bot/description/ros2_control.xacro (robot description, xacro)
@@ -1,25 +1,45 @@
-<ros2_control name="MyRobotSystem" type="system">
-  <hardware>
-    <plugin>gazebo_ros2_control/GazeboSystem</plugin>
-  </hardware>
-  <joint name="front_left_wheel_joint">
-    <command_interface name="velocity"/>
-    <state_interface name="velocity"/>
-    <state_interface name="position"/>
-  </joint>
-  <joint name="front_right_wheel_joint">
-    <command_interface name="velocity"/>
-    <state_interface name="velocity"/>
-    <state_interface name="position"/>
-  </joint>
-  <joint name="back_left_wheel_joint">
-    <command_interface name="velocity"/>
-    <state_interface name="velocity"/>
-    <state_interface name="position"/>
-  </joint>
-  <joint name="back_right_wheel_joint">
-    <command_interface name="velocity"/>
-    <state_interface name="velocity"/>
-    <state_interface name="position"/>
-  </joint>
-</ros2_control>
+<?xml version="1.0"?>
+<robot xmlns:xacro="http://www.ros.org/wiki/xacro">
+    <ros2_control name="GazeboSystem" type="system">
+        <hardware>
+            <plugin>gazebo_ros2_control/GazeboSystem</plugin>
+        </hardware>
+        <joint name="back_left_wheel_joint">
+            <command_interface name="velocity">
+                <param name ="min">-10</param>
+                <param name ="max">10</param>
+            </command_interface>
+            <state_interface name = "velocity"/>
+            <state_interface name = "position" />
+        </joint>
+        <joint name="back_right_wheel_joint">
+            <command_interface name="velocity">
+                <param name ="min">-10</param>
+                <param name ="max">10</param>
+            </command_interface>
+            <state_interface name = "velocity"/>
+            <state_interface name = "position" />
+        </joint>
+        <joint name="front_right_wheel_joint">
+            <command_interface name="velocity">
+                <param name ="min">-10</param>
+                <param name ="max">10</param>
+            </command_interface>
+            <state_interface name = "velocity"/>
+            <state_interface name = "position" />
+        </joint>
+        <joint name="front_left_wheel_joint">
+            <command_interface name="velocity">
+                <param name ="min">-10</param>
+                <param name ="max">10</param>
+            </command_interface>
+            <state_interface name = "velocity"/>
+            <state_interface name = "position" />
+        </joint>
+    </ros2_control>
+    <gazebo>
+        <plugin name="gazebo_ros2_control" filename="libgazebo_ros2_control.so">
+            <parameters>$(find my_bot)/config/my_controllers.yaml</parameters>
+        </plugin>
+    </gazebo>
+</robot>
