Commit message: ros2_control and SLAM

File: src/my_bot/description/lidar.xacro (robot description, xacro)
@@ -4,5 +4,5 @@
         <parent link="chassis"/>
         <child link="laser_frame"/>
-        <origin xyz="0.1 0 0.05" rpy="0 0 0"/>
+        <origin xyz="0.1 0 0.25" rpy="0 0 0"/>
     </joint>
     <link name="laser_frame">

File: src/my_bot/description/robot.urdf.xacro (robot description, xacro)
@@ -3,4 +3,5 @@
     <xacro:include filename="robot_core.xacro" />
     <xacro:include filename="inertial_macros.xacro" />
+    <xacro:include filename="lidar.xacro" />
     <xacro:include filename="ros2_control.xacro" />
 </robot>

File: src/my_bot/description/robot_core.xacro (robot description, xacro)
@@ -19,4 +19,12 @@
     <!-- BASE LINK -->
     <link name="base_link">
+    </link>
+    <!-- BASE_FOOTPRINT LINK -->
+    <joint name="base_footprint_joint" type="fixed">
+        <parent link="base_link"/>
+        <child link="base_footprint"/>
+        <origin xyz="0 0 0" rpy="0 0 0"/>
+    </joint>
+    <link name="base_footprint">
     </link>
     <!-- CHASSIS LINK -->
@@ -72,4 +80,6 @@
     <gazebo reference="left_wheel">
         <material>Gazebo/Blue</material>
+        <mu1 value="5.0"/>
+        <mu2 value="5.0"/>
     </gazebo>
     <!-- RIGHT WHEEL LINK -->
@@ -98,4 +108,6 @@
     <gazebo reference="right_wheel">
         <material>Gazebo/Blue</material>
+        <mu1 value="5.0"/>
+        <mu2 value="5.0"/>
     </gazebo>
     <!-- RIGHT FRONT WHEEL LINK -->
@@ -124,4 +136,6 @@
     <gazebo reference="right_front_wheel">
         <material>Gazebo/Blue</material>
+        <mu1 value="5.0"/>
+        <mu2 value="5.0"/>
     </gazebo>
     <!-- LEFT FRONT WHEEL LINK -->
@@ -150,4 +164,6 @@
     <gazebo reference="left_front_wheel">
         <material>Gazebo/Blue</material>
+       <mu1 value="5.0"/>
+        <mu2 value="5.0"/>
     </gazebo>
     <!-- IMU LINK -->
