Commit message: my_bot hardware interface

File: src/my_bot/description/ros2_control.xacro (robot description, xacro)
@@ -1,5 +1,51 @@
 <?xml version="1.0"?>
 <robot xmlns:xacro="http://www.ros.org/wiki/xacro">
-    <ros2_control name="GazeboSystem" type="system">
+    <ros2_control name="RealRobot" type="system">
+        <hardware>
+            <plugin>mecanumdrive_arduino/MecDriveArduinoHardware</plugin>
+            <param name="front_left_wheel_name">front_left_wheel_joint</param>
+            <param name="front_right_wheel_name">front_right_wheel_joint</param>
+            <param name="back_left_wheel_name">back_left_wheel_joint</param>
+            <param name="back_right_wheel_name">back_right_wheel_joint</param>
+            <param name="loop_rate">30</param>
+            <param name="device">/dev/ttyACM0</param>
+            <param name="baud_rate">57600</param>
+            <param name="timeout_ms">1000</param>
+            <param name="enc_counts_per_rev">3436</param>
+        </hardware>
+        <joint name="back_left_wheel_joint">
+            <command_interface name="velocity">
+                <param name ="min">-10</param>
+                <param name ="max">10</param>
+            </command_interface>
+            <state_interface name = "position" />
+            <state_interface name = "velocity"/>
+        </joint>
+        <joint name="back_right_wheel_joint">
+            <command_interface name="velocity">
+                <param name ="min">-10</param>
+                <param name ="max">10</param>
+            </command_interface>
+            <state_interface name = "position" />
+            <state_interface name = "velocity"/>
+        </joint>
+        <joint name="front_right_wheel_joint">
+            <command_interface name="velocity">
+                <param name ="min">-10</param>
+                <param name ="max">10</param>
+            </command_interface>
+            <state_interface name = "position" />
+            <state_interface name = "velocity"/>
+        </joint>
+        <joint name="front_left_wheel_joint">
+            <command_interface name="velocity">
+                <param name ="min">-10</param>
+                <param name ="max">10</param>
+            </command_interface>
+            <state_interface name = "position" />
+            <state_interface name = "velocity"/>
+        </joint>
+    </ros2_control>
+    <!-- <ros2_control name="GazeboSystem" type="system">
         <hardware>
             <plugin>gazebo_ros2_control/GazeboSystem</plugin>
@@ -37,5 +83,5 @@
             <state_interface name = "position" />
         </joint>
-    </ros2_control>
+    </ros2_control> -->
     <gazebo>
         <plugin name="gazebo_ros2_control" filename="libgazebo_ros2_control.so">
